File: case/plate/lk56hs-plate.kicad_pcb (KiCad board)
At the start: 2 copper layers, 247.7 x 95.2 mm, 53 parts

Commit message: Make plate reversible and add graphics
Parts:
- removed H1: MountingHole, LKBD_MountingHole:MountingHole_M2Head
- removed H3, H4, H6: MountingHole, LKBD_MountingHole:MountingSlot_M2Head_Small
- removed the REF** at (39.7, 54.0)
- removed the REF** at (87.3, 73.0)
- removed the REF** at (258.8, 54.0)
- removed the REF** at (106.4, 73.0)
- removed the REF** at (220.7, 73.0)
- removed the REF** at (161.2, 111.1)
- removed the REF** at (125.4, 73.0)
- removed the REF** at (42.1, 73.0)
- removed the REF** at (54.0, 34.9)
- removed the REF** at (201.6, 73.0)
- removed the REF** at (34.9, 34.9)
- removed the REF** at (182.6, 73.0)
- removed the REF** at (163.5, 73.0)
- removed the REF** at (144.5, 73.0)
- removed the REF** at (68.3, 73.0)
- added REF**: ClearanceHole_M2, LKBD_MountingHole:MountingHole_M2Head, F.Cu at (149.2, 63.5)
- added REF**: ClearanceHole_M2, LKBD_MountingHole:MountingHole_M2Head, F.Cu at (77.8, 101.6)
- added REF**: Plate_MX_2U_2x1U, LKBD_PlateMX:Plate_MX_2U_2x1U, B.Cu at (44.5, 34.9)
- added REF**: Plate_MX_1.5U, LKBD_PlateMX:Plate_MX_1.5U, B.Cu at (39.7, 54.0)
- added REF**: ClearanceHole_M2, LKBD_MountingHole:MountingHole_M2Head, F.Cu at (234.9, 82.5)
- added REF**: Plate_MX_2.25U_1U+1.25U, LKBD_PlateMX:Plate_MX_2.25U_1U+1.25U, B.Cu at (46.8, 73.0)
- added REF**: ClearanceHole_M2, LKBD_MountingHole:MountingHole_M2Head, F.Cu at (82.5, 44.5)
- added REF**: Plate_MX_1.5U, LKBD_PlateMX:Plate_MX_1.5U, B.Cu at (258.8, 54.0)
- added REF**: ClearanceHole_M2, LKBD_MountingHole:MountingHole_M2Head, F.Cu at (220.7, 101.6)
- added REF**: ClearanceHole_M2, LKBD_MountingHole:MountingHole_M2Head, F.Cu at (149.2, 82.5)
- added REF**: ClearanceHole_M2, LKBD_MountingHole:MountingHole_M2Head, F.Cu at (63.5, 82.5)
- added REF**: ClearanceHole_M2, LKBD_MountingHole:MountingHole_M2Head, F.Cu at (215.9, 44.5)
- REF** (x34): moved to B.Cu
- turned REF** to 180 degrees (x3)
- turned REF** to 0 degrees (x3)
Routing:
- added copper zone on F.Cu, net (none)
Other:
- outline, holes or cut-outs redrawn
