File: pcb/lk56hs-pcb.kicad_pcb (KiCad board)
At the start: 2 copper layers, 247.7 x 95.2 mm, 150 parts, among them J2 Conn_01x03, J3 Conn_01x05, SW1 RotaryEncoder_Switch_MP, SW10 SW_Push, SW11 SW_Push, SW12 SW_Push, SW13 SW_Push, SW14 SW_Push, SW15 SW_Push, SW16 SW_Push, SW17 SW_Push, SW18 SW_Push, SW19 SW_Push, SW2 SW_Push, SW20 SW_Push, SW21 SW_Push, SW22 SW_Push, SW23 SW_Push, SW24 SW_Push, SW25 SW_Push, SW26 SW_Push, SW27 SW_Push, SW28 SW_Push, SW29 SW_Push, SW3 SW_Push, SW30 SW_Push, SW31 SW_Push, SW32 SW_Push, SW33 SW_Push, SW34 SW_Push, SW35 SW_Push, SW36 SW_Push, SW37 SW_Push, SW38 SW_Push, SW39 SW_Push, SW4 SW_Push, SW40 SW_Push, SW41 SW_Push, SW42 SW_Push, SW43 SW_Push, SW44 SW_Push, SW45 SW_Push, SW46 SW_Push, SW47 SW_Push, SW48 SW_Push, SW49 SW_Push, SW5 SW_Push, SW50 SW_Push, SW51 SW_Push, SW52 SW_Push, SW53 SW_Push, SW54 SW_Push, SW55 SW_Push, SW56 SW_Push, SW57 SW_Push, SW58 SW_Push, SW59 SW_Push, SW6 SW_Push, SW60 SW_Push, SW61 SW_Push, SW62 SW_Push, SW63 SW_Push, SW64 SW_Push, SW65 SW_Push, SW66 SW_Push, SW67 SW_Push, SW68 SW_Push, SW69 SW_Push, SW7 SW_Push, SW70 SW_Push, SW71 SW_Push, SW8 SW_Push, SW9 SW_Push, U1 RaspberryPi_Pico

Commit message: Make plate reversible and add graphics
Parts:
- removed the H2 at (25.4, 101.6)
- added H3: MountingHole, LKBD_MountingHole:MountingHole_M2_NoPad, F.Cu at (149.2, 63.5)
- added H7: MountingHole, LKBD_MountingHole:MountingHole_M2_NoPad, F.Cu at (77.8, 101.6)
- added H8: MountingHole, LKBD_MountingHole:MountingHole_M2_NoPad, F.Cu at (220.7, 101.6)
- H1: footprint LKBD_MountingHole:MountingHole_M2_NPTH -> LKBD_MountingHole:MountingHole_M2_NoPad
- H2: renamed from H3; footprint LKBD_MountingHole:MountingSlot_M2_Small_NPTH -> LKBD_MountingHole:MountingHole_M2_NoPad
- H4, H6: footprint LKBD_MountingHole:MountingSlot_M2_Small_NPTH -> LKBD_MountingHole:MountingHole_M2_NoPad
- H5: footprint LKBD_MountingHole:MountingSlot_M2_NTPH_Long -> LKBD_MountingHole:MountingHole_M2_NoPad
- J2: value Conn_01x03 -> PINHD_1x03_ARGB
- J3: value Conn_01x05 -> PINHD_1x05_I2C
- moved H4 158.3 mm to (63.5, 82.5)
- moved H5 42.6 mm to (234.9, 82.5)
- moved H2 19.0 mm to (215.9, 44.5)
- moved H6 14.3 mm to (149.2, 82.5)
Other:
- outline, holes or cut-outs redrawn
