File: pcb/lk56hs-switch.kicad_sch (KiCad schematic)
At the start: 140 parts, among them SW1 RotaryEncoder_Switch_MP, SW10 SW_Push, SW11 SW_Push, SW12 SW_Push, SW13 SW_Push, SW14 SW_Push, SW15 SW_Push, SW16 SW_Push, SW17 SW_Push, SW18 SW_Push, SW19 SW_Push, SW2 SW_Push, SW20 SW_Push, SW21 SW_Push, SW22 SW_Push, SW23 SW_Push, SW24 SW_Push, SW25 SW_Push, SW26 SW_Push, SW27 SW_Push, SW28 SW_Push, SW29 SW_Push, SW3 SW_Push, SW30 SW_Push, SW31 SW_Push, SW32 SW_Push, SW33 SW_Push, SW34 SW_Push, SW35 SW_Push, SW36 SW_Push, SW37 SW_Push, SW38 SW_Push, SW39 SW_Push, SW4 SW_Push, SW40 SW_Push, SW41 SW_Push, SW42 SW_Push, SW43 SW_Push, SW44 SW_Push, SW45 SW_Push, SW46 SW_Push, SW47 SW_Push, SW48 SW_Push, SW49 SW_Push, SW5 SW_Push, SW50 SW_Push, SW51 SW_Push, SW52 SW_Push, SW53 SW_Push, SW54 SW_Push, SW55 SW_Push, SW56 SW_Push, SW57 SW_Push, SW58 SW_Push, SW59 SW_Push, SW6 SW_Push, SW60 SW_Push, SW61 SW_Push, SW62 SW_Push, SW63 SW_Push, SW64 SW_Push, SW65 SW_Push, SW66 SW_Push, SW67 SW_Push, SW68 SW_Push, SW69 SW_Push, SW7 SW_Push, SW70 SW_Push, SW71 SW_Push, SW8 SW_Push, SW9 SW_Push

Commit message: Update stabilizers
Parts:
- S13, S41, S53: footprint marbastlib-mx:STAB_MX_2u -> LKBD_StabMX:Stabilizer_MX_2U
- S38, S64: footprint marbastlib-mx:STAB_MX_2.25u -> LKBD_StabMX:Stabilizer_MX_2U
- S62: footprint marbastlib-mx:STAB_MX_2.75u -> LKBD_StabMX:Stabilizer_MX_2U
- S63: footprint marbastlib-mx:STAB_MX_6u -> LKBD_StabMX:Stabilizer_MX_6U
Changed lines of the file:
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@@
 			)
 		)
-		(property "Footprint" "marbastlib-mx:STAB_MX_2u"
+		(property "Footprint" "LKBD_StabMX:Stabilizer_MX_2U"
 			(at 10.16 107.95 0)
 			(effects
@@
 			)
 		)
-		(property "Footprint" "marbastlib-mx:STAB_MX_2.75u"
+		(property "Footprint" "LKBD_StabMX:Stabilizer_MX_2U"
 			(at 121.92 147.32 0)
 			(effects
@@
 			)
 		)
-		(property "Footprint" "marbastlib-mx:STAB_MX_2.25u"
+		(property "Footprint" "LKBD_StabMX:Stabilizer_MX_2U"
 			(at 287.02 88.9 0)
 			(effects
@@
 			)
 		)
-		(property "Footprint" "marbastlib-mx:STAB_MX_2u"
+		(property "Footprint" "LKBD_StabMX:Stabilizer_MX_2U"
 			(at 287.02 41.91 0)
 			(effects
@@
 			)
 		)
-		(property "Footprint" "marbastlib-mx:STAB_MX_2.25u"
+		(property "Footprint" "LKBD_StabMX:Stabilizer_MX_2U"
 			(at 165.1 147.32 0)
 			(effects
@@
 			)
 		)
-		(property "Footprint" "marbastlib-mx:STAB_MX_6u"
+		(property "Footprint" "LKBD_StabMX:Stabilizer_MX_6U"
 			(at 143.51 147.32 0)
 			(effects
@@
 			)
 		)
-		(property "Footprint" "marbastlib-mx:STAB_MX_2u"
+		(property "Footprint" "LKBD_StabMX:Stabilizer_MX_2U"
 			(at 287.02 107.95 0)
 			(effects

Commit message: Make plate reversible and add graphics
Changed lines of the file:
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@@
+	)
+	(junction
+		(at 60.96 127)
+		(diameter 0)
+		(color 0 0 0 0)
 	)
 	(junction
@@
 	)
 	(junction
+		(at 100.33 127)
+		(diameter 0)
+		(color 0 0 0 0)
+	)
+	(junction
 		(at 135.89 115.57)
 		(diameter 0)
@@
 		(diameter 0)
 		(color 0 0 0 0)
+	)
+	(junction
+		(at 153.67 127)
+		(diameter 0)
+		(color 0 0 0 0)

Commit message: Fix CPL output
Parts:
- SW55, SW56, SW57, SW58, SW59, SW60, SW61, SW63, SW65, SW66, SW67, SW68, SW69, SW70, SW71: JLCPosOffset -0.635,-3.81 -> 0.635,3.81
Changed lines of the file:
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@@
 			)
 		)
-		(property "JLCPosOffset" "-0.635,-3.81"
+		(property "JLCPosOffset" "0.635,3.81"
 			(at 219.71 127 0)
 			(effects
@@
 			)
 		)
-		(property "JLCPosOffset" "-0.635,-3.81"
+		(property "JLCPosOffset" "0.635,3.81"
 			(at 95.25 127 0)
 			(effects
@@
 			)
 		)
-		(property "JLCPosOffset" "-0.635,-3.81"
+		(property "JLCPosOffset" "0.635,3.81"
 			(at 201.93 127 0)
 			(effects
@@
 			)
 		)
-		(property "JLCPosOffset" "-0.635,-3.81"
+		(property "JLCPosOffset" "0.635,3.81"
 			(at 259.08 127 0)
 			(effects
@@
 			)
 		)
-		(property "JLCPosOffset" "-0.635,-3.81"
+		(property "JLCPosOffset" "0.635,3.81"
 			(at 148.59 127 0)
 			(effects
@@
 			)
 		)
-		(property "JLCPosOffset" "-0.635,-3.81"
+		(property "JLCPosOffset" "0.635,3.81"
 			(at 229.87 127 0)
 			(effects
@@
 			)
 		)
-		(property "JLCPosOffset" "-0.635,-3.81"
+		(property "JLCPosOffset" "0.635,3.81"
 			(at 105.41 127 0)
 			(effects
@@
 			)
 		)
-		(property "JLCPosOffset" "-0.635,-3.81"
+		(property "JLCPosOffset" "0.635,3.81"
 			(at 77.47 127 0)
 			(effects
@@
 			)
 		)
-		(property "JLCPosOffset" "-0.635,-3.81"
+		(property "JLCPosOffset" "0.635,3.81"
 			(at 66.04 127 0)
 			(effects
@@
 			)
 		)
-		(property "JLCPosOffset" "-0.635,-3.81"
+		(property "JLCPosOffset" "0.635,3.81"
 			(at 55.88 127 0)
 			(effects
@@
 			)
 		)
-		(property "JLCPosOffset" "-0.635,-3.81"
+		(property "JLCPosOffset" "0.635,3.81"
 			(at 241.3 127 0)
 			(effects
@@
 			)
 		)
-		(property "JLCPosOffset" "-0.635,-3.81"
+		(property "JLCPosOffset" "0.635,3.81"
 			(at 34.29 127 0)
 			(effects
@@
 			)
 		)
-		(property "JLCPosOffset" "-0.635,-3.81"
+		(property "JLCPosOffset" "0.635,3.81"
 			(at 191.77 127 0)
 			(effects
@@
 			)
 		)
-		(property "JLCPosOffset" "-0.635,-3.81"
+		(property "JLCPosOffset" "0.635,3.81"
 			(at 44.45 127 0)
 			(effects
@@
 			)
 		)
-		(property "JLCPosOffset" "-0.635,-3.81"
+		(property "JLCPosOffset" "0.635,3.81"
 			(at 269.24 127 0)
 			(effects
